File: Hardware/CAP1203.sch (EAGLE design)
At the start: 26 parts, among them J1 Qwiic Right Angle, J2 Qwiic Right Angle, J3 Cap Touch Breakout Pins, J4 I2C Breakout Pins, U2 CAP1203

Commit message: Added CAP1203 from SparkFun library
* Replaced current CAP1203 with SparkFun library version
* Updated in both sch and brd files
Parts:
- U2: device SparkX:CAP1203 -> SparkFun-Sensors:CAP1203
Changed lines of the file:
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@@
 <part name="SUPPLY6" library="SparkFun-PowerSymbols" deviceset="3.3V" device=""/>
 <part name="GND7" library="SparkFun-PowerSymbols" deviceset="GND" device=""/>
-<part name="U2" library="SparkX" deviceset="CAP1203" device="" value="CAP1203"/>
+<part name="U2" library="SparkFun-Sensors" deviceset="CAP1203" device="" value="CAP1203"/>
 <part name="JP3" library="SparkFun-Jumpers" deviceset="JUMPER-SMT_3_2-NC_TRACE" device="_SILK" value="JUMPER-SMT_3_2-NC_TRACE_SILK"/>
 <part name="R4" library="SparkFun-Resistors" deviceset="2.2KOHM" device="-0603-1/10W-1%" value="2.2k"/>
