File: Hardware/Production/CAP1203-Panel.brd (EAGLE design)
At the start: 96.8 x 97.3 mm, 264 parts, among them J1 Qwiic Right Angle, J10 Qwiic Right Angle, J11 Cap Touch Breakout Pins, J12 I2C Breakout Pins, J13 Qwiic Right Angle, J14 Qwiic Right Angle, J15 Cap Touch Breakout Pins, J16 I2C Breakout Pins, J17 Qwiic Right Angle, J18 Qwiic Right Angle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

Commit message: Removed extraneous files
Parts:
- U$100, U$32, U$49, U$66, U$83: value QWIIC_LOGO_5MM -> (none); device SparkFun-Aesthetics:QWIIC_5MM -> buzzard_labels (5):ACT0
- U$101, U$33, U$50, U$67, U$84: value QWIIC_LOGO_5MM -> (none); device SparkFun-Aesthetics:QWIIC_5MM -> buzzard_labels (10):CAPACITIVE_TOUCH_SLIDER0
- U$102, U$34, U$51, U$68, U$85: device buzzard_labels (5):ACT0 -> buzzard_labels (12):CAPACITIVE_TOUCH_SLIDER0
- U$18: device Labels:3V3-04 -> buzzard_labels (10):CAPACITIVE_TOUCH_SLIDER0
- U$19: device Labels:GND-04 -> buzzard_labels (12):CAPACITIVE_TOUCH_SLIDER0
- U$27, U$44, U$61, U$78, U$95: device buzzard_labels_title:CAPACITIVE_TOUCH_SLIDER0 -> Labels:I_SUPER2_C-()-03
- U$28, U$45, U$62, U$79, U$96: device buzzard_labels_title:CAPACITIVE_TOUCH_SLIDER0 -> buzzard_labels (4):INT0
- U$29, U$46, U$63, U$80, U$97: device Labels:I_SUPER2_C-()-03 -> Labels:PWR-()-03
- U$3: device buzzard_labels_title:CAPACITIVE_TOUCH_SLIDER0 -> Labels:3V3-04
- U$30, U$47, U$64, U$81, U$98: value (none) -> QWIIC_LOGO_5MM; device buzzard_labels (4):INT0 -> SparkFun-Aesthetics:QWIIC_5MM
- U$31, U$48, U$65, U$82, U$99: value (none) -> QWIIC_LOGO_5MM; device Labels:PWR-()-03 -> SparkFun-Aesthetics:QWIIC_5MM
- U$5: device buzzard_labels_title:CAPACITIVE_TOUCH_SLIDER0 -> Labels:GND-04
- U1, U2, U3, U4, U5, U6: device SparkX:SO08 -> SparkFun-Sensors:SO08-TIGHT
- moved U$3 63.3 mm to (70.5, 15.2)
- moved U$19 56.8 mm to (14.2, 8.38)
- moved U$18 40.8 mm to (30.2, 22.1), flipped to the bottom
- moved U$5 39.6 mm to (70.2, 17.8), flipped to the top
- moved U$45 23.4 mm to (8.51, 38.6), flipped to the top
- moved U$62 23.4 mm to (47.1, 38.6), flipped to the top
- moved U$28 23.4 mm to (47.1, 12.7), flipped to the top
- moved U$79 23.4 mm to (8.51, 64.5), flipped to the top
- moved U$96 23.4 mm to (47.1, 64.5), flipped to the top
- moved U$29 20.9 mm to (67.8, 19.9)
- moved U$46 20.9 mm to (29.2, 45.8)
- moved U$63 20.9 mm to (67.8, 45.8)
- moved U$80 20.9 mm to (29.2, 71.8)
- moved U$97 20.9 mm to (67.8, 71.8)
- moved LOGO20 19.7 mm to (21.1, 54.2)
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Routing:
- net CS13: track 38.4 -> 30.3 mm
- net CS16: track 38.4 -> 30.3 mm
- net CS4: track 38.4 -> 30.3 mm
- net CS10: track 38.4 -> 30.3 mm
- net CS7: track 38.4 -> 30.3 mm
- net CS1: track 38.4 -> 30.3 mm
- net CS8: track 24.3 -> 16.5 mm, vias 2 -> 1
- net CS2: track 24.3 -> 16.5 mm, vias 2 -> 1
- net CS11: track 24.3 -> 16.5 mm, vias 2 -> 1
- net CS5: track 24.3 -> 16.5 mm, vias 2 -> 1
- net CS14: track 24.3 -> 16.5 mm, vias 2 -> 1
- net CS17: track 24.3 -> 16.5 mm, vias 2 -> 1
- net 3.3V: track 67.1 -> 62.6 mm
- net 3.3V5: track 67.1 -> 62.6 mm
- net 3.3V4: track 67.1 -> 62.6 mm
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Other:
- board text added: "v10"
- board text removed: "x01"
